File: hardware/pcb/analogControlBoardV1.brd (EAGLE design)
At the start: 50 x 35 mm, 74 parts, among them IC1 OP07CR, IC2 OP07CR, IC3 4052D, IC4 741G53DCT, IC5 OP07CR, IC6 OP27D, IC7 AD633R, IC8 741G53DCT, U1 MAX6070, U2 MAX5216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

Commit message: analog version update
Parts:
- added TRIM: (no value), pinhead:1X02
Connections:
- net GND: now also TRIM.1
- net MULT_OUTPUT: now also TRIM.2
Routing:
- net MULT_OUTPUT: track 19.6 -> 35.4 mm, vias 2 -> 3
- net GND: vias 37 -> 35
- net -15V: vias 10 -> 9
- net +5V: vias 10 -> 9
- net +15V: vias 7 -> 6
Changed lines of the file:
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@@
 <layer number="23" name="tOrigins" color="15" fill="1" visible="yes" active="yes"/>
 <layer number="24" name="bOrigins" color="15" fill="1" visible="yes" active="yes"/>
-<layer number="25" name="tNames" color="7" fill="1" visible="no" active="yes"/>
+<layer number="25" name="tNames" color="7" fill="1" visible="yes" active="yes"/>
 <layer number="26" name="bNames" color="7" fill="1" visible="no" active="yes"/>
 <layer number="27" name="tValues" color="7" fill="1" visible="no" active="yes"/>
@@
 </element>
 <element name="R25" library="resistor" package="RTRIM64W" value="50k" x="32.7025" y="2.8575" smashed="yes" rot="R270">
-<attribute name="NAME" x="27.5425" y="2.67" size="0.8128" layer="25" font="vector" rot="R90"/>
+<attribute name="NAME" x="27.5425" y="3.94" size="0.8128" layer="25" font="vector" rot="R90"/>
 <attribute name="VALUE" x="27.7525" y="-1.4925" size="1.27" layer="27"/>
 </element>
@@
 <attribute name="NAME" x="13.0025" y="14.1225" size="0.8128" layer="25" font="vector" rot="R90"/>
 <attribute name="VALUE" x="14.35" y="11.5825" size="1.016" layer="27" rot="R90"/>
+</element>
+<element name="TRIM" library="pinhead" package="1X02" value="" x="25.0825" y="1.905" smashed="yes">
+<attribute name="NAME" x="22.4663" y="3.7338" size="1.27" layer="25" font="vector" ratio="10"/>
+<attribute name="VALUE" x="22.5425" y="-1.27" size="1.27" layer="27"/>
 </element>
 </elements>
@@
 <wire x1="35.2425" y1="1.5875" x2="35.2425" y2="6.6675" width="0.8128" layer="1"/>
 <wire x1="35.2425" y1="6.6675" x2="35.2425" y2="11.7475" width="0.8128" layer="1"/>
-<wire x1="40.64" y1="33.02" x2="40.64" y2="32.385" width="1.016" layer="1"/>
+<wire x1="40.64" y1="33.02" x2="40.64" y2="32.385" width="1.016" layer="16"/>
 <wire x1="40.64" y1="32.385" x2="36.5125" y2="28.2575" width="1.016" layer="16"/>
 <via x="14.9225" y="28.2575" extent="1-16" drill="0.3048" shape="octagon"/>
@@
 <wire x1="37.7825" y1="18.415" x2="35.56" y2="16.1925" width="0.6096" layer="1"/>
 <wire x1="35.56" y1="16.1925" x2="35.56" y2="15.24" width="0.6096" layer="1"/>
-<via x="40.64" y="32.385" extent="1-16" drill="0.3048" shape="octagon"/>
 </signal>
 <signal name="-15V">
@@
 <wire x1="30.1625" y1="1.5875" x2="30.1625" y2="6.6675" width="0.8128" layer="1"/>
 <wire x1="30.1625" y1="6.6675" x2="30.1625" y2="11.7475" width="0.8128" layer="1"/>
-<wire x1="35.56" y1="33.02" x2="35.56" y2="32.0675" width="1.016" layer="1"/>
+<wire x1="35.56" y1="33.02" x2="35.56" y2="32.0675" width="1.016" layer="16"/>
 <wire x1="35.56" y1="32.0675" x2="34.29" y2="30.7975" width="1.016" layer="16"/>
 <wire x1="34.29" y1="30.7975" x2="28.575" y2="30.7975" width="1.016" layer="16"/>
@@
 <wire x1="29.21" y1="18.0975" x2="29.21" y2="12.7" width="0.6096" layer="1"/>
 <wire x1="29.21" y1="12.7" x2="30.1625" y2="11.7475" width="0.6096" layer="1"/>
-<via x="35.56" y="32.0675" extent="1-16" drill="0.3048" shape="octagon"/>
 </signal>
 <signal name="GND">
@@
 <contactref element="U3" pad="4"/>
 <contactref element="U3" pad="8"/>
-<wire x1="33.02" y1="33.02" x2="29.845" y2="33.02" width="1.016" layer="16"/>
+<wire x1="33.02" y1="33.02" x2="29.845" y2="33.02" width="1.016" layer="1"/>
 <wire x1="29.845" y1="33.02" x2="26.035" y2="33.02" width="1.016" layer="1"/>
 <wire x1="26.035" y1="33.02" x2="25.4225" y2="33.02" width="1.016" layer="1"/>
@@
 <wire x1="16.1925" y1="25.9325" x2="16.1925" y2="32.9975" width="0.6096" layer="1"/>
 <wire x1="40.4" y1="24.13" x2="39.37" y2="24.13" width="0.6096" layer="1"/>
-<wire x1="39.37" y1="24.13" x2="33.02" y2="30.48" width="0.6096" layer="1"/>
-<wire x1="33.02" y1="30.48" x2="33.02" y2="33.02" width="0.6096" layer="16"/>
+<wire x1="33.02" y1="30.48" x2="33.02" y2="33.02" width="0.6096" layer="1"/>
 <wire x1="14.2875" y1="16.75" x2="15.875" y2="16.75" width="0.6096" layer="1"/>
 <wire x1="11.645" y1="20.955" x2="11.7475" y2="20.8525" width="0.6096" layer="1"/>
@@
 </polygon>
 <via x="31.115" y="33.02" extent="1-16" drill="0.3048" shape="octagon"/>
-<via x="29.845" y="33.02" extent="1-16" drill="0.3048" shape="octagon"/>
 <via x="43.18" y="33.02" extent="1-16" drill="0.3048" shape="octagon"/>
 <via x="48.26" y="28.575" extent="1-16" drill="0.3048" shape="octagon"/>
@@
 <via x="1.905" y="27.305" extent="1-16" drill="0.3048" shape="octagon"/>
 <via x="9.525" y="31.115" extent="1-16" drill="0.3048" shape="octagon"/>
-<via x="33.02" y="30.48" extent="1-16" drill="0.3048" shape="octagon"/>
+<contactref element="TRIM" pad="1"/>
+<wire x1="39.37" y1="24.13" x2="33.02" y2="30.48" width="0.6096" layer="1"/>
 </signal>
 <signal name="+5V">
@@
 <wire x1="14.2875" y1="12.5984" x2="14.2875" y2="13.97" width="0.6096" layer="1"/>
 <wire x1="14.2875" y1="13.97" x2="14.2875" y2="15" width="0.6096" layer="1"/>
-<wire x1="38.1" y1="33.02" x2="38.1" y2="32.385" width="1.016" layer="1"/>
+<wire x1="38.1" y1="33.02" x2="38.1" y2="32.385" width="1.016" layer="16"/>
 <wire x1="38.1" y1="32.385" x2="35.56" y2="29.845" width="1.016" layer="16"/>
 <via x="20.955" y="29.5275" extent="1-16" drill="0.3048" shape="octagon"/>
@@
 <wire x1="14.2875" y1="13.97" x2="20.32" y2="20.0025" width="1.016" layer="16"/>
 <wire x1="20.32" y1="20.0025" x2="20.32" y2="26.035" width="1.016" layer="16"/>
-<via x="38.1" y="32.385" extent="1-16" drill="0.3048" shape="octagon"/>
 </signal>
 <signal name="/CS2">
@@
 <wire x1="23.8125" y1="9.8425" x2="24.345" y2="10.375" width="0.4064" layer="1"/>
 <wire x1="24.345" y1="10.375" x2="24.765" y2="10.375" width="0.4064" layer="1"/>
+<contactref element="TRIM" pad="2"/>
+<wire x1="26.3525" y1="1.905" x2="26.9875" y2="2.54" width="0.4064" layer="1"/>
+<wire x1="26.9875" y1="2.54" x2="26.9875" y2="15.5575" width="0.4064" layer="1"/>
+<via x="26.9875" y="15.5575" extent="1-16" drill="0.3048" shape="octagon"/>
+<wire x1="26.9875" y1="15.5575" x2="25.0825" y2="15.5575" width="0.4064" layer="16"/>
 </signal>
 <signal name="N$38">
