File: hardware/pcb/analogBoardV1_5.brd (EAGLE design)
At the start: 100 x 50 mm, 76 parts, among them IC1 74AC139D, IC3 741G53DCT, IC4 MEGA8-AI, IC6 LM35DT, IC7 LM35DT, Q1 IRFP250, Q10 BSS123, Q2 IRFP250, Q3 IRFP250, Q4 IRFP250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

Commit message: cleaned up schematics + markings an analogBoard
Connections:
- net N$9 renamed FET_GATE
Routing:
- net FET_GATE: track 175.2 -> 176.0 mm
Other:
- board text added: "+15"
- board text added: "+5"
- board text added: "-15"
- board text added: "AnalogBoard V1.5"
- board text added: "CS_A"
- board text added: "CS_B"
- board text added: "DIN"
- board text added: "DOUT1"
- board text added: "DOUT2"
- board text added: "ElectronicLoad"
- board text added: "GND"
- board text added: "INPUT"
- board text added: "SCLK"
- board text added: "github.com/jankae/electronicload"
