File: hardware/pcb/analogBoardV1_5.sch (EAGLE design)
At the start: 76 parts, among them IC1 74AC139D, IC3 741G53DCT, IC4 MEGA8-AI, IC6 LM35DT, IC7 LM35DT, Q1 IRFP250, Q10 BSS123, Q2 IRFP250, Q3 IRFP250, Q4 IRFP250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

Commit message: cleaned up schematics + markings an analogBoard
Connections:
- net N$9 renamed FET_GATE
Other:
- note added: "FET driver"
- note added: "analog control board connection"
- note added: "glue logic"
- note added: "input protection, power stage and shunt resistors"
- note added: "isolated interface"
- note added: "power"
- note added: "temperature measurement"
- moved on the sheet: B1, C1, C10, C11, C12, C2, C3, C5, C6, C7, C8, D1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
