File: hardware/pcb/analogControlBoardV1.sch (EAGLE design)
At the start: 74 parts, among them IC1 OP07CR, IC2 OP07CR, IC3 4052D, IC4 741G53DCT, IC5 OP07CR, IC6 OP27D, IC7 AD633R, IC8 741G53DCT, U1 MAX6070, U2 MAX5216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

Commit message: analog version update
Parts:
- added TRIM: (no value), pinhead:PINHD-1X2
Connections:
- net GND: now also TRIM.1
- net MULT_OUTPUT: now also TRIM.2
Changed lines of the file:
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@@
 <part name="P-9" library="supply1" deviceset="-15V" device=""/>
 <part name="GND13" library="supply1" deviceset="GND" device=""/>
+<part name="TRIM" library="pinhead" deviceset="PINHD-1X2" device=""/>
+<part name="GND17" library="supply1" deviceset="GND" device=""/>
 </parts>
 <sheets>
@@
 <instance part="P-9" gate="1" x="215.9" y="426.72" rot="MR180"/>
 <instance part="GND13" gate="1" x="205.74" y="406.4"/>
+<instance part="TRIM" gate="G$1" x="355.6" y="254" rot="MR180"/>
+<instance part="GND17" gate="1" x="345.44" y="246.38"/>
 </instances>
 <busses>
@@
 <junction x="205.74" y="411.48"/>
 </segment>
+<segment>
+<pinref part="TRIM" gate="G$1" pin="1"/>
+<wire x1="353.06" y1="251.46" x2="345.44" y2="251.46" width="0.1524" layer="91"/>
+<wire x1="345.44" y1="251.46" x2="345.44" y2="248.92" width="0.1524" layer="91"/>
+<pinref part="GND17" gate="1" pin="GND"/>
+</segment>
 </net>
 <net name="+5V" class="0">
@@
 <junction x="281.94" y="287.02"/>
 </segment>
-</net>
+<segment>
+<pinref part="TRIM" gate="G$1" pin="2"/>
+<wire x1="353.06" y1="254" x2="345.44" y2="254" width="0.1524" layer="91"/>
+<label x="345.44" y="254" size="1.778" layer="95" rot="R180" xref="yes"/>
+</segment>
+</net>

Commit message: cleaned up schematics + markings an analogBoard
Other:
- note added: "ADC+mux"
- note added: "DAC"
- note added: "central control OP-amp with mux"
- note added: "connectors"
- note added: "current/voltage sensing"
- note added: "decoupling"
- note added: "mulitplier stage"
- note added: "offset compensation for multiplier"
- note removed: "current setting DAC"
- note removed: "voltage and current amplifier"
- note removed: "voltage/current ADC"
- moved on the sheet: 4.096V, C1, C10, C11, C12, C13, C14, C15, C16, C17, C18, C19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
